Commit message: feat: redesign URDF model with simplified meshes and enhance debugger
- Replace part-level meshes with joint-level naming (l1-l6, jaw, el05_l6)
- Remove legacy EL_A3_urdf directory
- Add motor calibration feature (calibration_worker, calibration_panel)
- Enhance debugger UI: i18n, 3D viewer, diagnostics panel
- Update ROS2 xacro/joint_limits configuration
- Update SDK interface

Made-with: Cursor

File: el_a3_ros/EDULITE-A3/EDULITE-A3.urdf (robot description, URDF)
Before this commit: robot EDULITE-A3, 7 links, 6 joints
Links:
- removed link l1_link_urdf_asm
- removed link l1_urdf_urdf_asm
- removed link l2_l3_urdf_asm
- removed link l3_lnik_urdf_asm
- removed link l4_l5_urdf_asm
- removed link l5_l6_urdf_asm
- removed link part_9
- added link l1_link_urdf_asm_copy_1, mass 0.105244; collision mesh filename=package://meshes/l2.stl; visual mesh filename=package://meshes/l2.stl
- added link l1_urdf_urdf_asm_copy_1, mass 0.498832; collision mesh filename=package://meshes/l1.stl; visual mesh filename=package://meshes/l1.stl
- added link l2_l3_urdf_asm_copy_1, mass 0.836196; collision mesh filename=package://meshes/l3.stl; visual mesh filename=package://meshes/l3.stl
- added link l3_lnik_urdf_asm_copy_1, mass 0.262025; collision mesh filename=package://meshes/l4.stl; visual mesh filename=package://meshes/l4.stl
- added link l4_l5_urdf_asm_copy_1, mass 0.55715; collision mesh filename=package://meshes/l5.stl; visual mesh filename=package://meshes/l5.stl
- added link l5_l6_urdf_asm_copy_1, mass 0.657292; collision mesh filename=package://meshes/el05_l6.stl; collision mesh filename=package://meshes/jaw.stl
- added link l6, mass 0.0392349; collision mesh filename=package://meshes/l6.stl; visual mesh filename=package://meshes/l6.stl
Joints:
- joint L1_joint: axis 0 0 1 -> 0 0 -1; child l1_link_urdf_asm -> l1_link_urdf_asm_copy_1; origin xyz=0 0 0.006 rpy=0 -0 0 -> xyz=-4.9779e-07 -1.62314e-10 0.06 rpy=3.14159 -5.8976e-28 2.77556e-17; parent l1_urdf_urdf_asm -> l1_urdf_urdf_asm_copy_1
- joint L2_joint: child l2_l3_urdf_asm -> l2_l3_urdf_asm_copy_1; origin xyz=-0.01 -0.0006 0.064 rpy=1.5708 -0 9.72346e-63 -> xyz=-0.00964286 3.46945e-18 -0.069 rpy=-1.5708 -0 1.30819e-41; parent l1_link_urdf_asm -> l1_link_urdf_asm_copy_1
- joint L3_joint: child l3_lnik_urdf_asm -> l3_lnik_urdf_asm_copy_1; limit lower=-4.01426 upper=0 effort=10 velocity=10 -> lower=-4.01426 upper=-0 effort=10 velocity=10; origin xyz=0.19 1.249e-16 0.0518 rpy=2.54281e-17 7.99959e-17 8.37004e-17 -> xyz=0.19 -2.77556e-17 -2.76776e-18 rpy=-9.46633e-29 -2.78912e-28 3.72342e-28; parent l2_l3_urdf_asm -> l2_l3_urdf_asm_copy_1
- joint L4_joint: axis 0 0 1 -> 0 0 -1; child l4_l5_urdf_asm -> l4_l5_urdf_asm_copy_1; limit lower=-1.5708 upper=1.5708 effort=10 velocity=10 -> lower=-1.0472 upper=1.5708 effort=10 velocity=10; origin xyz=-0.185 0.064 -0.0518 rpy=2.5974e-22 2.98284e-23 -4.33681e-19 -> xyz=-0.185 0.064 6.93889e-18 rpy=-3.14159 1.18102e-27 3.88578e-16; parent l3_lnik_urdf_asm -> l3_lnik_urdf_asm_copy_1
- joint L5_joint: child part_9 -> l6; origin xyz=-0.0492 0.038 5.24537e-16 rpy=1.5708 -1.89036e-16 1.56125e-17 -> xyz=-0.0492 -0.038 5.95508e-17 rpy=-1.5708 1.13007e-27 3.88578e-16; parent l4_l5_urdf_asm -> l4_l5_urdf_asm_copy_1
- joint L6_joint: child l5_l6_urdf_asm -> l5_l6_urdf_asm_copy_1; origin xyz=0.00805 -2.47957e-16 0.038 rpy=-1.5708 -5.60446e-32 -1.5708 -> xyz=0.00685 -2.9256e-16 0.039 rpy=-1.5708 -0 -1.5708; parent part_9 -> l6

File: el_a3_ros/el_a3_description/urdf/el_a3.urdf (robot description, URDF)
Before this commit: robot EL-A3, 10 links, 9 joints
Links:
- link l1_link_urdf_asm: mass 0.146738 -> 0.105244; geometry collision mesh filename=package://el_a3_description/meshes/l2.stl; visual mesh filename=package://el_a3_description/meshes/l2.stl
- link l1_urdf_urdf_asm: mass 0.465144 -> 0.498832; geometry collision mesh filename=package://el_a3_description/meshes/l1.stl; visual mesh filename=package://el_a3_description/meshes/l1.stl
- link l2_l3_urdf_asm: mass 0.946534 -> 0.836196; geometry collision mesh filename=package://el_a3_description/meshes/l3.stl; visual mesh filename=package://el_a3_description/meshes/l3.stl
- link l3_lnik_urdf_asm: mass 0.406558 -> 0.262025; geometry collision mesh filename=package://el_a3_description/meshes/l4.stl; visual mesh filename=package://el_a3_description/meshes/l4.stl
- link l4_l5_urdf_asm: mass 0.54692 -> 0.55715; geometry collision mesh filename=package://el_a3_description/meshes/l5.stl; visual mesh filename=package://el_a3_description/meshes/l5.stl
- link l5_l6_urdf_asm: mass 0.6317 -> 0.657292; geometry collision mesh filename=package://el_a3_description/meshes/el05_l6.stl; collision mesh filename=package://el_a3_description/meshes/jaw.stl
- link part_9: mass 0.031 -> 0.0392349; geometry collision mesh filename=package://el_a3_description/meshes/l6.stl; visual mesh filename=package://el_a3_description/meshes/l6.stl
Joints:
- joint L1_joint: axis 0 0 1 -> 0 0 -1; origin xyz=0 0 0.006 rpy=0 0 0 -> xyz=0 0 0.06 rpy=3.14159 0 0
- joint L2_joint: origin xyz=-0.01 -0.0006 0.064 rpy=1.5708 0 0 -> xyz=-0.00964286 0 -0.069 rpy=-1.5708 0 0
- joint L3_joint: origin xyz=0.19 0 0.0518 rpy=0 0 0 -> xyz=0.19 0 0 rpy=0 0 0
- joint L4_joint: axis 0 0 1 -> 0 0 -1; limit lower=-1.5708 upper=1.5708 effort=6.0 velocity=50 -> lower=-1.0472 upper=1.5708 effort=6.0 velocity=50; origin xyz=-0.185 0.064 -0.0518 rpy=0 0 0 -> xyz=-0.185 0.064 0 rpy=-3.14159 0 0
- joint L5_joint: origin xyz=-0.0492 0.038 0 rpy=1.5708 0 0 -> xyz=-0.0492 -0.038 0 rpy=-1.5708 0 0
- joint L6_joint: origin xyz=0.00805 0 0.038 rpy=-1.5708 0 -1.5708 -> xyz=0.00685 0 0.039 rpy=-1.5708 0 -1.5708

File: el_a3_ros/el_a3_description/urdf/el_a3.urdf.xacro (robot description, xacro)
@@ -17,24 +17,6 @@
     <color rgba="0.972549 0.529412 0.00392157 1"/>
   </material>
-  <material name="gray">
-    <color rgba="0.647059 0.647059 0.647059 1"/>
-  </material>
-  <material name="light_blue">
-    <color rgba="0.768627 0.886275 0.952941 1"/>
-  </material>
-  <material name="white">
-    <color rgba="0.917647 0.917647 0.917647 1"/>
-  </material>
-  <material name="dark_gray">
-    <color rgba="0.301961 0.301961 0.301961 1"/>
-  </material>
-  <material name="blue">
-    <color rgba="0.231373 0.380392 0.705882 1"/>
-  </material>
-  <material name="yellow">
-    <color rgba="0.980392 0.713725 0.00392157 1"/>
-  </material>
-  <material name="green">
-    <color rgba="0.372549 0.654902 0.239216 1"/>
+  <material name="dark_brown">
+    <color rgba="0.301961 0.290196 0.262745 1"/>
   </material>
   <!-- Base link (world) -->
@@ -48,35 +30,20 @@
   <link name="l1_urdf_urdf_asm">
     <inertial>
-      <origin xyz="-2.68984e-10 1.48294e-05 -0.0220571" rpy="0 0 0"/>
-      <mass value="0.465144"/>
-      <inertia ixx="0.00032748" ixy="-1.33894e-08" ixz="-1.85358e-12"
-               iyy="0.000321793" iyz="-2.46949e-07" izz="0.000362426"/>
-    </inertial>
-    <!-- Part part_10 -->
-    <visual>
-      <origin xyz="0 0 0" rpy="0 0 0"/>
-      <geometry>
-        <mesh filename="package://el_a3_description/meshes/part_10.stl"/>
-      </geometry>
-      <material name="green"/>
-    </visual>
-    <collision>
-      <origin xyz="0 0 0" rpy="0 0 0"/>
-      <geometry>
-        <mesh filename="package://el_a3_description/meshes/part_10.stl"/>
-      </geometry>
-    </collision>
-    <!-- Part rs00_l1 -->
-    <visual>
-      <origin xyz="0 0 0" rpy="0 0 0"/>
-      <geometry>
-        <mesh filename="package://el_a3_description/meshes/rs00_l1.stl"/>
-      </geometry>
-      <material name="orange"/>
-    </visual>
-    <collision>
-      <origin xyz="0 0 0" rpy="0 0 0"/>
-      <geometry>
-        <mesh filename="package://el_a3_description/meshes/rs00_l1.stl"/>
+      <origin xyz="4.66057e-08 7.85527e-05 0.0336468" rpy="0 0 0"/>
+      <mass value="0.498832"/>
+      <inertia ixx="0.000371872" ixy="-1.33362e-08" ixz="5.96807e-10"
+               iyy="0.000365137" iyz="-1.36721e-06" izz="0.000388475"/>
+    </inertial>
+    <visual>
+      <origin xyz="-0.000643355 0 0.059" rpy="0 0 0"/>
+      <geometry>
+        <mesh filename="package://el_a3_description/meshes/l1.stl"/>
+      </geometry>
+      <material name="dark_brown"/>
+    </visual>
+    <collision>
+      <origin xyz="-0.000643355 0 0.059" rpy="0 0 0"/>
+      <geometry>
+        <mesh filename="package://el_a3_description/meshes/l1.stl"/>
       </geometry>
     </collision>
@@ -85,35 +52,20 @@
   <link name="l1_link_urdf_asm">
     <inertial>
-      <origin xyz="-0.00202103 -0.00162495 0.0394318" rpy="0 0 0"/>
-      <mass value="0.146738"/>
-      <inertia ixx="0.000221617" ixy="-1.44161e-06" ixz="1.46922e-05"
-               iyy="0.000129193" iyz="4.22954e-06" izz="0.000175411"/>
-    </inertial>
-    <!-- Part part_8 -->
-    <visual>
-      <origin xyz="0 0 -0.006" rpy="0 0 0"/>
-      <geometry>
-        <mesh filename="package://el_a3_description/meshes/part_8.stl"/>
-      </geometry>
-      <material name="yellow"/>
-    </visual>
-    <collision>
-      <origin xyz="0 0 -0.006" rpy="0 0 0"/>
-      <geometry>
-        <mesh filename="package://el_a3_description/meshes/part_8.stl"/>
-      </geometry>
-    </collision>
-    <!-- Part part_9 -->
-    <visual>
-      <origin xyz="0 0 -0.006" rpy="0 0 0"/>
-      <geometry>
-        <mesh filename="package://el_a3_description/meshes/part_9.stl"/>
-      </geometry>
-      <material name="yellow"/>
-    </visual>
-    <collision>
-      <origin xyz="0 0 -0.006" rpy="0 0 0"/>
-      <geometry>
-        <mesh filename="package://el_a3_description/meshes/part_9.stl"/>
+      <origin xyz="-0.00232762 -0.00161986 0.0421389" rpy="0 0 0"/>
+      <mass value="0.105244"/>
+      <inertia ixx="0.000163151" ixy="-3.25924e-06" ixz="1.01303e-05"
+               iyy="9.80821e-05" iyz="1.04567e-05" izz="0.000118753"/>
+    </inertial>
+    <visual>
+      <origin xyz="-0.000642857 0 0.001" rpy="3.14159 0 0"/>
+      <geometry>
+        <mesh filename="package://el_a3_description/meshes/l2.stl"/>
+      </geometry>
+      <material name="orange"/>
+    </visual>
+    <collision>
+      <origin xyz="-0.000642857 0 0.001" rpy="3.14159 0 0"/>
+      <geometry>
+        <mesh filename="package://el_a3_description/meshes/l2.stl"/>
       </geometry>
     </collision>
@@ -122,91 +74,20 @@
   <link name="l2_l3_urdf_asm">
     <inertial>
-      <origin xyz="0.0949994 -1.38262e-06 -0.00108795" rpy="0 0 0"/>
-      <mass value="0.946534"/>
-      <inertia ixx="0.000493341" ixy="6.92125e-07" ixz="-1.27006e-08"
-               iyy="0.00767087" iyz="2.73309e-09" izz="0.0076934"/>
-    </inertial>
-    <!-- Part mainlink_back -->
-    <visual>
-      <origin xyz="0.01 -0.07 -0.0001" rpy="-1.5708 0 0"/>
-      <geometry>
-        <mesh filename="package://el_a3_description/meshes/mainlink_back.stl"/>
-      </geometry>
-      <material name="gray"/>
-    </visual>
-    <collision>
-      <origin xyz="0.01 -0.07 -0.0001" rpy="-1.5708 0 0"/>
-      <geometry>
-        <mesh filename="package://el_a3_description/meshes/mainlink_back.stl"/>
-      </geometry>
-    </collision>
-    <!-- Part 6705 -->
-    <visual>
-      <origin xyz="0.01 -0.07 -0.0001" rpy="-1.5708 0 0"/>
-      <geometry>
-        <mesh filename="package://el_a3_description/meshes/6705.stl"/>
-      </geometry>
-      <material name="white"/>
-    </visual>
-    <collision>
-      <origin xyz="0.01 -0.07 -0.0001" rpy="-1.5708 0 0"/>
-      <geometry>
-        <mesh filename="package://el_a3_description/meshes/6705.stl"/>
-      </geometry>
-    </collision>
-    <!-- Part rs00_l2 -->
-    <visual>
-      <origin xyz="0.01 -0.07 -0.0006" rpy="-1.5708 0 0"/>
-      <geometry>
-        <mesh filename="package://el_a3_description/meshes/rs00_l2.stl"/>
-      </geometry>
-      <material name="orange"/>
-    </visual>
-    <collision>
-      <origin xyz="0.01 -0.07 -0.0006" rpy="-1.5708 0 0"/>
-      <geometry>
-        <mesh filename="package://el_a3_description/meshes/rs00_l2.stl"/>
-      </geometry>
-    </collision>
-    <!-- Part mainlink_motor -->
-    <visual>
-      <origin xyz="0.01 -0.07 -0.0006" rpy="-1.5708 0 0"/>
-      <geometry>
-        <mesh filename="package://el_a3_description/meshes/mainlink_motor.stl"/>
-      </geometry>
-      <material name="gray"/>
-    </visual>
-    <collision>
-      <origin xyz="0.01 -0.07 -0.0006" rpy="-1.5708 0 0"/>
-      <geometry>
-        <mesh filename="package://el_a3_description/meshes/mainlink_motor.stl"/>
-      </geometry>
-    </collision>
-    <!-- Part 6705_2 -->
-    <visual>
-      <origin xyz="0.01 -0.07 -0.0001" rpy="-1.5708 0 0"/>
-      <geometry>
-        <mesh filename="package://el_a3_description/meshes/6705__2.stl"/>
-      </geometry>
-      <material name="blue"/>
-    </visual>
-    <collision>
-      <origin xyz="0.01 -0.07 -0.0001" rpy="-1.5708 0 0"/>
-      <geometry>
-        <mesh filename="package://el_a3_description/meshes/6705__2.stl"/>
-      </geometry>
-    </collision>
-    <!-- Part rs00_l3 -->
-    <visual>
-      <origin xyz="0.01 -0.07 -0.0006" rpy="-1.5708 0 0"/>
-      <geometry>
-        <mesh filename="package://el_a3_description/meshes/rs00_l3.stl"/>
-      </geometry>
-      <material name="orange"/>
-    </visual>
-    <collision>
-      <origin xyz="0.01 -0.07 -0.0006" rpy="-1.5708 0 0"/>
-      <geometry>
-        <mesh filename="package://el_a3_description/meshes/rs00_l3.stl"/>
+      <origin xyz="0.0949957 1.32911e-06 0.000626283" rpy="0 0 0"/>
+      <mass value="0.836196"/>
+      <inertia ixx="0.000419405" ixy="-4.27021e-07" ixz="-4.05336e-10"
+               iyy="0.00708317" iyz="2.8291e-09" izz="0.00707892"/>
+    </inertial>
+    <visual>
+      <origin xyz="0.009 -0.07 0" rpy="-1.5708 0 0"/>
+      <geometry>
+        <mesh filename="package://el_a3_description/meshes/l3.stl"/>
+      </geometry>
+      <material name="dark_brown"/>
+    </visual>
+    <collision>
+      <origin xyz="0.009 -0.07 0" rpy="-1.5708 0 0"/>
+      <geometry>
+        <mesh filename="package://el_a3_description/meshes/l3.stl"/>
       </geometry>
     </collision>
@@ -215,35 +96,20 @@
   <link name="l3_lnik_urdf_asm">
     <inertial>
-      <origin xyz="-0.0693243 0.0530595 -0.0510805" rpy="0 0 0"/>
-      <mass value="0.406558"/>
-      <inertia ixx="0.000554036" ixy="0.000274809" ixz="4.74842e-06"
-               iyy="0.00189339" iyz="7.79959e-06" izz="0.00192037"/>
-    </inertial>
-    <!-- Part small_arm_right -->
-    <visual>
-      <origin xyz="-0.18 -0.07 -0.0518" rpy="-1.5708 0 0"/>
-      <geometry>
-        <mesh filename="package://el_a3_description/meshes/small_arm_right.stl"/>
-      </geometry>
-      <material name="orange"/>
-    </visual>
-    <collision>
-      <origin xyz="-0.18 -0.07 -0.0518" rpy="-1.5708 0 0"/>
-      <geometry>
-        <mesh filename="package://el_a3_description/meshes/small_arm_right.stl"/>
-      </geometry>
-    </collision>
-    <!-- Part small_arm_left -->
-    <visual>
-      <origin xyz="-0.18 -0.07 -0.0518" rpy="-1.5708 0 0"/>
-      <geometry>
-        <mesh filename="package://el_a3_description/meshes/small_arm_left.stl"/>
-      </geometry>
-      <material name="orange"/>
-    </visual>
-    <collision>
-      <origin xyz="-0.18 -0.07 -0.0518" rpy="-1.5708 0 0"/>
-      <geometry>
-        <mesh filename="package://el_a3_description/meshes/small_arm_left.stl"/>
+      <origin xyz="-0.0743466 -0.0535452 -0.00326782" rpy="0 0 0"/>
+      <mass value="0.262025"/>
+      <inertia ixx="0.000333463" ixy="-0.000182996" ixz="-9.89508e-06"
+               iyy="0.00130159" iyz="1.18614e-05" izz="0.00133147"/>
+    </inertial>
+    <visual>
+      <origin xyz="-0.181 -0.07 0" rpy="-1.5708 0 0"/>
+      <geometry>
+        <mesh filename="package://el_a3_description/meshes/l4.stl"/>
+      </geometry>
+      <material name="orange"/>
+    </visual>
+    <collision>
+      <origin xyz="-0.181 -0.07 0" rpy="-1.5708 0 0"/>
+      <geometry>
+        <mesh filename="package://el_a3_description/meshes/l4.stl"/>
       </geometry>
     </collision>
@@ -252,77 +118,20 @@
   <link name="l4_l5_urdf_asm">
     <inertial>
-      <origin xyz="-0.0241077 0.0297756 -0.000254349" rpy="0 0 0"/>
-      <mass value="0.54692"/>
-      <inertia ixx="0.000543249" ixy="0.000320527" ixz="2.88671e-06"
-               iyy="0.00040341" iyz="-3.57587e-06" izz="0.000797799"/>
-    </inertial>
-    <!-- Part el05_l5 -->
-    <visual>
-      <origin xyz="0.005 -0.134 0" rpy="-1.5708 0 0"/>
-      <geometry>
-        <mesh filename="package://el_a3_description/meshes/el05_l5.stl"/>
-      </geometry>
-      <material name="white"/>
-    </visual>
-    <collision>
-      <origin xyz="0.005 -0.134 0" rpy="-1.5708 0 0"/>
-      <geometry>
-        <mesh filename="package://el_a3_description/meshes/el05_l5.stl"/>
-      </geometry>
-    </collision>
-    <!-- Part l5_shake -->
-    <visual>
-      <origin xyz="0.005 -0.134 0" rpy="-1.5708 0 0"/>
-      <geometry>
-        <mesh filename="package://el_a3_description/meshes/l5_shake.stl"/>
-      </geometry>
-      <material name="light_blue"/>
-    </visual>
-    <collision>
-      <origin xyz="0.005 -0.134 0" rpy="-1.5708 0 0"/>
-      <geometry>
-        <mesh filename="package://el_a3_description/meshes/l5_shake.stl"/>
-      </geometry>
-    </collision>
-    <!-- Part l4_l5_link_back -->
-    <visual>
-      <origin xyz="0.005 -0.134 0" rpy="-1.5708 0 0"/>
-      <geometry>
-        <mesh filename="package://el_a3_description/meshes/l4_l5_link_back.stl"/>
-      </geometry>
-      <material name="orange"/>
-    </visual>
-    <collision>
-      <origin xyz="0.005 -0.134 0" rpy="-1.5708 0 0"/>
-      <geometry>
-        <mesh filename="package://el_a3_description/meshes/l4_l5_link_back.stl"/>
-      </geometry>
-    </collision>
-    <!-- Part el05_l4 -->
-    <visual>
-      <origin xyz="0.005 -0.134 0" rpy="-1.5708 0 0"/>
-      <geometry>
-        <mesh filename="package://el_a3_description/meshes/el05_l4.stl"/>
-      </geometry>
-      <material name="white"/>
-    </visual>
-    <collision>
-      <origin xyz="0.005 -0.134 0" rpy="-1.5708 0 0"/>
-      <geometry>
-        <mesh filename="package://el_a3_description/meshes/el05_l4.stl"/>
-      </geometry>
-    </collision>
-    <!-- Part l4_l5_link_back_2 -->
-    <visual>
-      <origin xyz="0.005 -0.134 0" rpy="-1.5708 0 0"/>
-      <geometry>
-        <mesh filename="package://el_a3_description/meshes/l4_l5_link_back__2.stl"/>
-      </geometry>
-      <material name="orange"/>
-    </visual>
-    <collision>
-      <origin xyz="0.005 -0.134 0" rpy="-1.5708 0 0"/>
-      <geometry>
-        <mesh filename="package://el_a3_description/meshes/l4_l5_link_back__2.stl"/>
+      <origin xyz="-0.0242818 -0.0298393 0.000368105" rpy="0 0 0"/>
+      <mass value="0.55715"/>
+      <inertia ixx="0.0006785" ixy="-0.000401622" ixz="-5.0507e-06"
+               iyy="0.000503952" iyz="-6.21816e-06" izz="0.000993465"/>
+    </inertial>
+    <visual>
+      <origin xyz="0.004 0.134 0" rpy="1.5708 0 0"/>
+      <geometry>
+        <mesh filename="package://el_a3_description/meshes/l5.stl"/>
+      </geometry>
+      <material name="dark_brown"/>
+    </visual>
+    <collision>
+      <origin xyz="0.004 0.134 0" rpy="1.5708 0 0"/>
+      <geometry>
+        <mesh filename="package://el_a3_description/meshes/l5.stl"/>
       </geometry>
     </collision>
@@ -331,21 +140,20 @@
   <link name="part_9">
     <inertial>
-      <origin xyz="0.00409255 0 0.0175119" rpy="0 0 0"/>
-      <mass value="0.031"/>
-      <inertia ixx="5.21252e-06" ixy="0" ixz="-1.22446e-06"
-               iyy="5.09672e-06" iyz="0" izz="2.51083e-06"/>
-    </inertial>
-    <!-- Part part_9_2 -->
-    <visual>
-      <origin xyz="0.0542 0 0.172" rpy="3.14159 0 0"/>
-      <geometry>
-        <mesh filename="package://el_a3_description/meshes/part_9__2.stl"/>
-      </geometry>
-      <material name="orange"/>
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
File: el_a3_ros/el_a3_description/urdf/el_a3_ros2_control.xacro (robot description, xacro)
@@ -156,5 +156,5 @@
         <param name="zero_torque_kd_max">0.1</param>
         <command_interface name="position">
-          <param name="min">-1.5708</param>
+          <param name="min">-1.0472</param>
           <param name="max">1.5708</param>
         </command_interface>

File: el_a3_sdk/resources/rs05/urdf/el_a3.urdf (robot description, URDF)
Before this commit: robot EL-A3, 9 links, 8 joints
Links:
- link l1_link_urdf_asm: mass 0.146738 -> 0.105244; geometry collision mesh filename=package://el_a3_description/meshes/l2.stl; visual mesh filename=package://el_a3_description/meshes/l2.stl
- link l1_urdf_urdf_asm: mass 0.465144 -> 0.498832; geometry collision mesh filename=package://el_a3_description/meshes/l1.stl; visual mesh filename=package://el_a3_description/meshes/l1.stl
- link l2_l3_urdf_asm: mass 0.946534 -> 0.836196; geometry collision mesh filename=package://el_a3_description/meshes/l3.stl; visual mesh filename=package://el_a3_description/meshes/l3.stl
- link l3_lnik_urdf_asm: mass 0.406558 -> 0.262025; geometry collision mesh filename=package://el_a3_description/meshes/l4.stl; visual mesh filename=package://el_a3_description/meshes/l4.stl
- link l4_l5_urdf_asm: mass 0.44692 -> 0.55715; geometry collision mesh filename=package://el_a3_description/meshes/l5.stl; visual mesh filename=package://el_a3_description/meshes/l5.stl
- link l5_l6_urdf_asm: mass 0.5317 -> 0.657292; geometry collision mesh filename=package://el_a3_description/meshes/el05_l6.stl; collision mesh filename=package://el_a3_description/meshes/jaw.stl
- link part_9: mass 0.0179457 -> 0.0392349; geometry collision mesh filename=package://el_a3_description/meshes/l6.stl; visual mesh filename=package://el_a3_description/meshes/l6.stl
Joints:
- joint L1_joint: axis 0 0 1 -> 0 0 -1; origin xyz=0 0 0.006 rpy=0 0 0 -> xyz=0 0 0.06 rpy=3.14159 0 0
- joint L2_joint: origin xyz=-0.01 -0.0006 0.064 rpy=1.5708 0 0 -> xyz=-0.00964286 0 -0.069 rpy=-1.5708 0 0
- joint L3_joint: origin xyz=0.19 0 0.0518 rpy=0 0 0 -> xyz=0.19 0 0 rpy=0 0 0
- joint L4_joint: axis 0 0 1 -> 0 0 -1; limit lower=-1.5708 upper=1.5708 effort=6.0 velocity=50 -> lower=-1.0472 upper=1.5708 effort=6.0 velocity=50; origin xyz=-0.185 0.064 -0.0518 rpy=0 0 0 -> xyz=-0.185 0.064 0 rpy=-3.14159 0 0
- joint L5_joint: origin xyz=-0.0492 0.038 0 rpy=1.5708 0 0 -> xyz=-0.0492 -0.038 0 rpy=-1.5708 0 0
- joint L6_joint: origin xyz=0.00805 0 0.038 rpy=-1.5708 0 -1.5708 -> xyz=0.00685 0 0.039 rpy=-1.5708 0 -1.5708
