Commit message: feat: redesign URDF model with simplified meshes and enhance debugger
- Replace part-level meshes with joint-level naming (l1-l6, jaw, el05_l6)
- Remove legacy EL_A3_urdf directory
- Add motor calibration feature (calibration_worker, calibration_panel)
- Enhance debugger UI: i18n, 3D viewer, diagnostics panel
- Update ROS2 xacro/joint_limits configuration
- Update SDK interface

Made-with: Cursor

File: el_a3_sdk/resources/urdf/el_a3.urdf (robot description, URDF)
Before this commit: robot EL-A3, 10 links, 9 joints
Links:
- link l1_link_urdf_asm: mass 0.146738 -> 0.105244; geometry collision mesh filename=package://el_a3_description/meshes/l2.stl; visual mesh filename=package://el_a3_description/meshes/l2.stl
- link l1_urdf_urdf_asm: mass 0.465144 -> 0.498832; geometry collision mesh filename=package://el_a3_description/meshes/l1.stl; visual mesh filename=package://el_a3_description/meshes/l1.stl
- link l2_l3_urdf_asm: mass 0.946534 -> 0.836196; geometry collision mesh filename=package://el_a3_description/meshes/l3.stl; visual mesh filename=package://el_a3_description/meshes/l3.stl
- link l3_lnik_urdf_asm: mass 0.406558 -> 0.262025; geometry collision mesh filename=package://el_a3_description/meshes/l4.stl; visual mesh filename=package://el_a3_description/meshes/l4.stl
- link l4_l5_urdf_asm: mass 0.54692 -> 0.55715; geometry collision mesh filename=package://el_a3_description/meshes/l5.stl; visual mesh filename=package://el_a3_description/meshes/l5.stl
- link l5_l6_urdf_asm: mass 0.6317 -> 0.657292; geometry collision mesh filename=package://el_a3_description/meshes/el05_l6.stl; collision mesh filename=package://el_a3_description/meshes/jaw.stl
- link part_9: mass 0.031 -> 0.0392349; geometry collision mesh filename=package://el_a3_description/meshes/l6.stl; visual mesh filename=package://el_a3_description/meshes/l6.stl
Joints:
- joint L1_joint: axis 0 0 1 -> 0 0 -1; origin xyz=0 0 0.006 rpy=0 0 0 -> xyz=0 0 0.06 rpy=3.14159 0 0
- joint L2_joint: origin xyz=-0.01 -0.0006 0.064 rpy=1.5708 0 0 -> xyz=-0.00964286 0 -0.069 rpy=-1.5708 0 0
- joint L3_joint: origin xyz=0.19 0 0.0518 rpy=0 0 0 -> xyz=0.19 0 0 rpy=0 0 0
- joint L4_joint: axis 0 0 1 -> 0 0 -1; limit lower=-1.5708 upper=1.5708 effort=6.0 velocity=50 -> lower=-1.0472 upper=1.5708 effort=6.0 velocity=50; origin xyz=-0.185 0.064 -0.0518 rpy=0 0 0 -> xyz=-0.185 0.064 0 rpy=-3.14159 0 0
- joint L5_joint: origin xyz=-0.0492 0.038 0 rpy=1.5708 0 0 -> xyz=-0.0492 -0.038 0 rpy=-1.5708 0 0
- joint L6_joint: origin xyz=0.00805 0 0.038 rpy=-1.5708 0 -1.5708 -> xyz=0.00685 0 0.039 rpy=-1.5708 0 -1.5708
